Commit message: Initial support for Lidar sensors (#6)
* Updating test resources

* Initial setup of LiDAR sensors

* Parsing lidar data from config

* Publish lidar messages

* Update lidar example and get publish rates

* Minor cleanup

* Update rviz config

* Move the rangefinder

* Update documentation

* Only copy sensordata rather than all data

* Add a comment

* Transforms on the range

* Update test rviz config

* Add lidar conversion support and update the example robot

* Update src/mujoco_system_interface.cpp

Co-authored-by: Nathan Dunkelberger <138718889+ndunkelb-nasa@users.noreply.github.com>

* Name the image

* Add .gitignore

* Add rviz to the test deps

* Use a lidar tag and do all the frame conversion in the script

* Pull min and max angle from ros2 control xacro, don't assume min_angle is always 0

* Turn off rangefinder rendering in cameras

* Apply suggestions from code review

* Pre-commit fixes

* Add a node about lidar scan time

* Update class comment

* Set a default ROS_DOMAIN_ID just in case

---------

Co-authored-by: Nathan Dunkelberger <138718889+ndunkelb-nasa@users.noreply.github.com>

File: test/test_resources/test_robot.urdf (robot description, URDF)
Before this commit: robot two_dof_robot, 9 links, 8 joints
Links:
- added link lidar_sensor_frame
Joints:
- added joint lidar_sensor_link: type fixed, parent world, child lidar_sensor_frame, origin xyz=1.0 2.0 0 rpy=0 0 -1.5708

Commit message: Consolidate the URDFs for PID and non-PID control

File: test/test_resources/test_robot.urdf (robot description, URDF)
Before this commit: robot two_dof_robot, 10 links, 9 joints
Links:
- link forearm: mass 27.0 -> 1.0
- link upperarm: mass 27.0 -> 1.0

Commit message: fix masses in URDF to be similar to MJCF existing files

File: test/test_resources/test_robot.urdf (robot description, URDF)
Before this commit: robot two_dof_robot, 10 links, 9 joints
Links:
- link forearm: mass 1.0 -> 27.0
- link upperarm: mass 1.0 -> 27.0

Commit message: Add basic pjm to the test robot

File: test/test_resources/test_robot.urdf (robot description, URDF)
Before this commit: robot two_dof_robot, 10 links, 9 joints
Links:
- added link gripper_base, mass 0.5; collision box size=0.08 0.12 0.04; visual box size=0.08 0.12 0.04
- added link gripper_left_finger, mass 0.1; collision box size=0.02 0.01 0.1; visual box size=0.02 0.01 0.1
- added link gripper_right_finger, mass 0.1; collision box size=0.02 0.05 0.1; visual box size=0.02 0.01 0.1
Joints:
- added joint gripper_base_joint: type fixed, parent ee_link, child gripper_base, origin xyz=0.04 0 -0.02 rpy=0 1.5708 0
- added joint gripper_left_finger_joint: type prismatic, parent gripper_base, child gripper_left_finger, origin xyz=0 0.05 0 rpy=0 0 0, axis 0 1 0, limit lower=-0.045 upper=0.005 effort=50 velocity=0.1
- added joint gripper_right_finger_joint: type prismatic, parent gripper_base, child gripper_right_finger, origin xyz=0 -0.05 0 rpy=0 0 0, axis 0 1 0, limit lower=-0.005 upper=0.045 effort=50 velocity=0.1

Commit message: Mimic joint and fix control coeffs for the gripper

File: test/test_resources/test_robot.urdf (robot description, URDF)
Before this commit: robot two_dof_robot, 13 links, 12 joints
Joints:
- joint gripper_right_finger_joint: mimic (none) -> joint=gripper_left_finger_joint multiplier=-1 offset=0

Commit message: Added prismatic gripper to the test robot to validate tendons functionality (#64)
---------

Co-authored-by: Erik Holum <erik.holum@nasa.gov>
Co-authored-by: Nathan Dunkelberger <nathan.b.dunkelberger@nasa.gov>

File: test/test_resources/test_robot.urdf (robot description, URDF)
Before this commit: robot two_dof_robot, 10 links, 9 joints
Links:
- added link gripper_base, mass 0.5; collision box size=0.08 0.12 0.04; visual box size=0.08 0.12 0.04
- added link gripper_left_finger, mass 0.1; collision box size=0.02 0.01 0.1; visual box size=0.02 0.01 0.1
- added link gripper_right_finger, mass 0.1; collision box size=0.02 0.05 0.1; visual box size=0.02 0.01 0.1
Joints:
- added joint gripper_base_joint: type fixed, parent ee_link, child gripper_base, origin xyz=0.04 0 -0.02 rpy=0 1.5708 0
- added joint gripper_left_finger_joint: type prismatic, parent gripper_base, child gripper_left_finger, origin xyz=0 0.05 0 rpy=0 0 0, axis 0 1 0, limit lower=-0.045 upper=0.005 effort=50 velocity=0.1
- added joint gripper_right_finger_joint: type prismatic, parent gripper_base, child gripper_right_finger, origin xyz=0 -0.05 0 rpy=0 0 0, axis 0 1 0, limit lower=-0.005 upper=0.045 effort=50 velocity=0.1, mimic joint=gripper_left_finger_joint multiplier=-1 offset=0
