Commit message: Update demo robots

File: mujoco_ros2_control_demos/demo_resources/robot/test_robot.urdf (robot description, URDF)
Before this commit: robot two_dof_robot, 13 links, 12 joints
Links:
- added link 3d_lidar_sensor_frame
Joints:
- added joint 3d_lidar_sensor_link: type fixed, parent world, child 3d_lidar_sensor_frame, origin xyz=1.0 -2.0 0 rpy=0 0 1.5708

Commit message: Remove the lidar extension from the demos for now

File: mujoco_ros2_control_demos/demo_resources/robot/test_robot.urdf (robot description, URDF)
Before this commit: robot two_dof_robot, 14 links, 13 joints
Links:
- removed link 3d_lidar_sensor_frame
Joints:
- removed joint 3d_lidar_sensor_link
