Commit message: Simplify comments

File: mujoco_ros2_control_demos/demo_resources/mobile_base/mobile_base.urdf (robot description, URDF)
Before this commit: robot mobile_base, 3 links, 2 joints
Joints:
- removed joint base_footprint_joint
- added joint world_to_base_joint: type fixed, parent world, child base_link
